File: hw/carrier-board/output/sonde-carrier.kicad_pcb (KiCad board)
At the start: 2 copper layers, 25 x 35 mm, 16 parts

Commit message: fix: cargo fmt + remove leftover edited/ directory
Co-authored-by: Copilot <223556219+Copilot@users.noreply.github.com>
Other:
- rule pad_to_mask_clearance: 0.1 -> 0
Changed lines of the file:
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@@
 	)
 	(setup
-		(pad_to_mask_clearance 0.1)
-		(solder_mask_min_width 0.1)
+		(stackup
+			(layer "F.SilkS"
+				(type "Top Silk Screen")
+			)
+			(layer "F.Paste"
+				(type "Top Solder Paste")
+			)
+			(layer "F.Mask"
+				(type "Top Solder Mask")
+				(thickness 0.01)
+			)
+			(layer "F.Cu"
+				(type "copper")
+				(thickness 0.035)
+			)
+			(layer "dielectric 1"
+				(type "core")
+				(thickness 1.51)
+				(material "FR4")
+				(epsilon_r 4.5)
+				(loss_tangent 0.02)
+			)
+			(layer "B.Cu"
+				(type "copper")
+				(thickness 0.035)
+			)
+			(layer "B.Mask"
+				(type "Bottom Solder Mask")
+				(thickness 0.01)
+			)
+			(layer "B.Paste"
+				(type "Bottom Solder Paste")
+			)
+			(layer "B.SilkS"
+				(type "Bottom Silk Screen")
+			)
+			(copper_finish "None")
+			(dielectric_constraints no)
+		)
+		(pad_to_mask_clearance 0)
 		(allow_soldermask_bridges_in_footprints no)
 		(pcbplotparams
